File: hardware/rgbtime.kicad_pcb (KiCad board)
At the start: 2 copper layers, 50 x 50 mm, 53 parts, among them CON1 AVR-ISP-6, IC1 ATMEGA8-AI, IC10 WS2812B, IC11 WS2812B, IC12 WS2812B, IC13 WS2812B, IC14 WS2812B, IC15 WS2812B, IC16 WS2812B, IC17 WS2812B, IC18 WS2812B, IC19 WS2812B, IC2 WS2812B, IC20 WS2812B, IC21 WS2812B, IC22 WS2812B, IC23 WS2812B, IC24 WS2812B, IC25 WS2812B, IC26 WS2812B, IC3 WS2812B, IC4 WS2812B, IC5 WS2812B, IC6 WS2812B, IC7 WS2812B, IC8 WS2812B, IC9 WS2812B, P2 POWER, U1 MCP79410, U2 LM75, U3 LM317S, Y1 CC4V-T1A-32768

Commit message: final hardware revision A done, sent to fab
Parts:
- added G***: LOGO, LOGO, B.Cu at (164.0, 91.2)
Connections:
- IC1 pad 26: Net-(IC1-Pad26) -> /RTC_ALM
- IC1 pad 32: Net-(IC1-Pad32) -> /LM75_ALM
- U1 pad 7: Net-(U1-Pad7) -> /RTC_ALM
- U2 pad 3: Net-(U2-Pad3) -> /LM75_ALM
Routing:
- net /LM75_ALM: track 0.00 -> 25.7 mm, vias 0 -> 2
- net /RTC_ALM: track 0.00 -> 14.8 mm, vias 0 -> 2
