File: hardware/rgbtime.sch (KiCad schematic (older format))
At the start: 41 parts, among them CON1 AVR-ISP-6, IC1 ATMEGA8-AI, IC10 WS2812B, IC11 WS2812B, IC12 WS2812B, IC13 WS2812B, IC14 WS2812B, IC15 WS2812B, IC16 WS2812B, IC17 WS2812B, IC18 WS2812B, IC19 WS2812B, IC2 WS2812B, IC20 WS2812B, IC21 WS2812B, IC22 WS2812B, IC23 WS2812B, IC24 WS2812B, IC25 WS2812B, IC26 WS2812B, IC3 WS2812B, IC4 WS2812B, IC5 WS2812B, IC6 WS2812B, IC7 WS2812B, IC8 WS2812B, IC9 WS2812B, P1 USB-Mini-B, U1 MCP79410, U2 LM75, Y1 CC4V-T1A-32768

Commit message: restructured repo
Parts:
- removed P1: USB-Mini-B, symbol USB_OTG
- added C5, C6: C, Capacitors_SMD:C_0603_HandSoldering, symbol C
- added C7, C8: 1u, Capacitors_SMD:C_0805_HandSoldering, symbol C
- added P2: POWER, Connect:bornier2, symbol CONN_01X02
- added R6, R7: 330, Resistors_SMD:R_0603_HandSoldering, symbol R
- added R8: 220, Resistors_SMD:R_0603_HandSoldering, symbol R
- added U3: LM317S, SMD_Packages:TO-263, symbol LM317S
Connections:
- net labels added: B_CAP, P_IN, RTC_BACK
- net labels removed: RST
- wire segments 221 -> 235
- no-connect marks 25 -> 21
Other:
- moved on the sheet: C2, C3, C4, CON1, D1, R2, R3, R4, R5, U1, U2, Y1

Commit message: final hardware revision A done, sent to fab
Connections:
- net RTC_ALM: now reaches IC1.26 ((ADC3)PC3)
- net RTC_ALM: now also U1.7 (MFP)
- net LM75_ALM: now reaches IC1.32 ((INT0)PD2)
- net LM75_ALM: now also U2.3 (O.S.)
- no-connect marks 21 -> 17
